File: EscolleraCircuito/Escollera.kicad_pcb (KiCad board)
At the start: 2 copper layers, 12 parts, among them J1 Conn_01x02, J2 Conn_01x04, J3 Conn_01x04, U1 LM7812_TO220, U2 LM7805_TO220, U3 MAX485E, U4 MAX485E, U5 TTGO_LoRa32

Commit message: pdfs del esquemático y la PCB
Routing:
- removed copper zone on F.Cu, net GND
